File: pedometer.sch (EAGLE design)
At the start: 2 parts, among them U1 LSM6DSO32TRLGA-14L_2P5X3X0P83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

Commit message: COmpleted board files
Parts:
- added C1, C2: 0.1uF, SparkFun-Capacitors:0.1UF-0603-25V-(+80/-20%)
- added D1: BLUE, SparkFun-LED:LED-BLUE0603
- added J1: (no value), SparkFun-Connectors:CONN_05
- added J2: (no value), SparkFun-Connectors:QWIIC_CONNECTORJS-1MM
- added J3: 1012, 1012:1012
- added J4: (no value), SparkFun-Connectors:CONN_04
- added Q1: 2.5A/30V/105mΩ, SparkFun-DiscreteSemi:MOSFET_PCH-DMG2307L
- added R1, R2: 2.2k, SparkFun-Resistors:2.2KOHM-0603-1/10W-1%
- added R3: 220, SparkFun-Resistors:220OHM-0603-1/10W-1%
Connections:
- new net GND: C1.1, C2.1, H1.VSS/VSSA, J1.3, J2.1, J3.-_2, J4.VCC, Q1.G, U1.GND, U1.GND_2, U1.SDO/SA0
- new net INT1: H1.PA4, U1.INT1
- new net INT2: H1.PA5, U1.INT2
- new net N$1: J3.+_1, J3.-_1
- new net N$2: J3.+_2, Q1.D
- new net N$3: H1.PA3, R3.1
- new net N$4: D1.C, R3.2
- new net NRST: H1.PF2-NRST, J1.5
- new net SCL: H1.PA11[PA9], J2.4, J4.GND, R1.1, U1.SCL
- new net SDA: H1.PA12[PA10], J2.3, J4.SDA, R2.1, U1.SDA
- new net SWCLK: H1.PA15/PA14-BOOT0, J1.2
- new net SWDIO: H1.PA13, J1.4
- new net VDD: C1.2, C2.2, D1.A, H1.VDD/VDDA, J1.1, J2.2, J4.SCL, Q1.S, R1.2, R2.2, U1.CS, U1.VDD, U1.VDDIO
Other:
- moved on the sheet: U1
